Commit message: Add files via upload

File: rover1/urdf/rover2.xacro (robot description, xacro)
@@ -11,10 +11,10 @@
     <xacro:property name="orientation_part_1" value="${pi/2} 0 ${pi/2}"/>
     <xacro:property name="orientation_part_2" value="0 0 ${pi/2}"/>
-    <xacro:property name="wheel_rientation" value="0 0 ${pi/2}"/>
+    <xacro:property name="wheel_orientation" value="0 0 ${pi/2}"/>
     <link name="base_link">
         <inertial>
             <origin xyz="0.0 0.0 0.0" rpy="0.0 0.0 0.0"/>
             <mass value="60"/>
-            <inertia ixx="0.0" ixy="0.0" ixz="0.0" iyy="0.0" iyz="0.0" izz="0.0"/>
+            <inertia ixx="1.0" ixy="0.0" ixz="0.0" iyy="1.0" iyz="0.0" izz="1.0"/>
         </inertial>
         <visual >
@@ -87,5 +87,5 @@
                 <origin xyz="0.0 0.0 0.0" rpy="0.0 ${pi/2} ${pi/2}"/>
                 <geometry>
-                    <cylinder radius="${r}" length="${h}"/>
+                    <cylinder radius="${r}" length="${h/1.2}"/>
                 </geometry>
                 <material name="dark_blue">
@@ -96,5 +96,5 @@
                 <origin xyz="0.0 0.0 0.0" rpy="0.0 ${pi/2} ${pi/2}"/>
                 <geometry>
-                    <cylinder radius="${r}" length="${h}"/>
+                    <cylinder radius="${r}" length="${h/18}"/>
                 </geometry>
             </collision>
@@ -105,5 +105,5 @@
             <child link="${wheel_name}"/>
             <axis xyz="0 1 0"/>
-            <origin xyz="${-(wheel_support2_length/2)-0.03} 0 ${-(wheel_support1_length/2)}" rpy="${wheel_rientation}"/>
+            <origin xyz="${-(wheel_support2_length/2)-0.03} 0 ${-(wheel_support1_length/2)}" rpy="${wheel_orientation}"/>
             <limit effort="30.0" velocity="100.0"/>
         </joint>
@@ -113,5 +113,5 @@
             <child link="${name2}"/>
             <axis xyz="0 0 1"/>
-            <limit lower="-${pi}" upper="${pi}" effort="1.0" velocity="1.0"/>
+            <limit lower="-3.14" upper="3.14" effort="10.0" velocity="10.0"/>
         </joint>
         <joint name="${joint_support_motor}" type="fixed">
